File: hardware/FOC2.kicad_pcb (KiCad board)
At the start: 2 copper layers, 50 x 55 mm, 95 parts, among them J1 Conn_01x03, J2 Conn_01x02, J4 Conn_01x02, J6 Conn_01x04, J8 Conn_01x03, J9 Conn_01x04, Q1 Q_NMOS_SGD, Q2 Q_NMOS_SGD, Q3 Q_NMOS_SGD, Q4 Q_NMOS_SGD, Q5 Q_NMOS_SGD, Q6 Q_NMOS_SGD, U1 LM321, U10 REF3033, U3 STM32G431CBUx, U4 EG2133, U5 INA199xxDCK, U6 INA199xxDCK, U7 TPS54360DDA, U8 TJA1044GTK/3Z, U9 LP5907MFX-3.3

Commit message: feat : redesign
Parts:
- C17: footprint Library:C_1812_4532Metric -> Capacitor_SMD:C_1812_4532Metric
- C18, C19, C20, C21, C22, C23, C24, C25, C26, C27, C31, C32, C33, C34, C35, C36, C37, C38, C39, C5, C6, C7, C8: footprint Library:C_0603_1608Metric -> Capacitor_SMD:C_0603_1608Metric
- C28, C29: footprint Library:C_0603_1608Metric -> Capacitor_SMD:C_0603_1608Metric; moved to F.Cu
- D10, D11, D2: footprint Library:D_SOD-323_HandSoldering -> Diode_SMD:D_SOD-123
- D12: footprint Library:Nexperia_CFP3_SOD-123W -> Diode_SMD:Nexperia_CFP3_SOD-123W
- D13: footprint Library:LED_0603_1608Metric -> LED_SMD:LED_0603_1608Metric
- D3: footprint Library:D_SMA -> Diode_SMD:D_SMA
- D4, D5, D6, D7, D8, D9: footprint Library:D_SOD-123 -> Diode_SMD:D_SOD-123
- H1, H2, H3, H4: footprint Library:MountingHole_2.2mm_M2_DIN965_Pad -> MountingHole:MountingHole_2.2mm_M2_DIN965_Pad
- J1: footprint Library:AMASS_MR30PW-FB_1x03_P3.50mm_Horizontal -> Connector_AMASS:AMASS_MR30PW-FB_1x03_P3.50mm_Horizontal
- J4: footprint Library:AMASS_XT30PW-F_1x02_P2.50mm_Horizontal -> Connector_AMASS:AMASS_XT30PW-F_1x02_P2.50mm_Horizontal; moved to F.Cu
- L1: footprint Library:L_Abracon_ASPI-0630LR -> Inductor_SMD:L_Abracon_ASPI-0630LR
- Q1, Q2, Q3, Q4, Q5, Q6: footprint Library:VSONP-8-1EP_5x6_P1.27mm -> Package_SON:VSONP-8-1EP_5x6_P1.27mm
- R1, R12, R13, R14, R15, R16, R17, R18, R19, R2, R23, R24, R25, R26, R4, R5, R7, R8: footprint Library:R_0603_1608Metric -> Resistor_SMD:R_0603_1608Metric
- R11, R28, R29: moved to F.Cu
- R3, R6, R9: footprint Library:R_2512_6332Metric -> Resistor_SMD:R_2512_6332Metric
- U1: footprint Library:SOT-23-5 -> Package_TO_SOT_SMD:SOT-23-5; moved to F.Cu
- U10: footprint Library:SOT-23 -> Package_TO_SOT_SMD:SOT-23
- U3: footprint Library:QFN-48-1EP_7x7mm_P0.5mm_EP5.6x5.6mm -> Package_DFN_QFN:QFN-48-1EP_7x7mm_P0.5mm_EP5.6x5.6mm
- U4: footprint Library:TSSOP-20_4.4x6.5mm_P0.65mm -> Package_SO:TSSOP-20_4.4x6.5mm_P0.65mm
- U5, U6: footprint Library:SOT-363_SC-70-6 -> Package_TO_SOT_SMD:SOT-363_SC-70-6; moved to F.Cu
- U7: footprint Library:TI_SO-PowerPAD-8_ThermalVias -> Package_SO:TI_SO-PowerPAD-8_ThermalVias
- U8: footprint Library:HVSON-8-1EP_3x3mm_P0.65mm_EP1.6x2.4mm -> Package_SON:HVSON-8-1EP_3x3mm_P0.65mm_EP1.6x2.4mm
- U9: footprint Library:SOT-23-5 -> Package_TO_SOT_SMD:SOT-23-5
- moved L1 135.6 mm to (81.7, 79.4)
- moved C26 124.3 mm to (37.4, 79.1), turned to 0 degrees
- moved C27 123.4 mm to (37.4, 81.6), turned to 0 degrees
- moved R13 123.1 mm to (45.5, 79.1), turned to 0 degrees
- moved R14 122.5 mm to (45.5, 81.6), turned to 0 degrees
- moved C38 115.3 mm to (41.4, 79.1), turned to 0 degrees
- moved C17 114.4 mm to (82.8, 95.5), turned to 0 degrees
- moved R15 114.3 mm to (45.5, 84.1)
- moved C5 113.4 mm to (33.4, 76.6), turned to 0 degrees
- moved R16 113.4 mm to (45.5, 86.6), turned to 0 degrees
- moved C39 112.0 mm to (41.4, 81.6), turned to 0 degrees
- moved C6 111.3 mm to (33.4, 79.1), turned to 0 degrees
- moved C33 110.3 mm to (37.4, 94.1), turned to 0 degrees
- moved R26 110.3 mm to (49.5, 84.1)
- moved C7 110.2 mm to (33.4, 81.6), turned to 0 degrees
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Connections:
- C26 pad 1: +3.3V -> +3V3
- C27 pad 1: +3.3V -> +3V3
- C28 pad 1: +3.3V -> +3V3
- C29 pad 1: +3.3V -> +3V3
- C7 pad 1: +3.3V -> +3V3
- C8 pad 1: +3.3V -> +3V3
- R13 pad 2: +3.3V -> +3V3
- U1 pad 5: +3.3V -> +3V3
- U5 pad 3: +3.3V -> +3V3
- U6 pad 3: +3.3V -> +3V3
- U9 pad 5: +3.3V -> +3V3
Routing:
- net Earth: track 397.2 -> 0.00 mm
- net Net-(D5-A): track 27.2 -> 0.00 mm, vias 1 -> 0
- net Net-(D4-A): track 13.6 -> 0.00 mm
- net Net-(D8-A): track 13.4 -> 0.00 mm
- net Net-(D6-A): track 13.2 -> 0.00 mm
- net Net-(D7-A): track 6.56 -> 0.00 mm, vias 1 -> 0
- net /M1_SL_C: track 5.81 -> 0.00 mm, vias 2 -> 0
- net /M1_SL_B: track 5.68 -> 0.00 mm, vias 2 -> 0
- net GND: track 5.45 -> 0.00 mm, vias 39 -> 0
- net /VS3: track 4.70 -> 0.00 mm
- net /M1_SL_A: track 3.57 -> 0.00 mm, vias 1 -> 0
- net /M1_GH_B: track 2.73 -> 0.00 mm
- net /M1_GH_C: track 2.68 -> 0.00 mm
- net /M1_GH_A: track 2.67 -> 0.00 mm
- net /VS1: track 1.53 -> 0.00 mm
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- removed copper zone on F.Cu, net /M1_SL_A
- removed copper zone on F.Cu, net /M1_SL_B
- removed copper zone on F.Cu, net /M1_SL_C
- removed copper zone on F.Cu, net /VS1
- removed copper zone on F.Cu, net /VS2
- removed copper zone on F.Cu, net /VS3
- removed copper zone on B.Cu, net GND
- removed copper zone on F.Cu, net GND
- removed copper zone on B.Cu, net VDC
- removed copper zone on F.Cu, net VDC
Other:
- board outline removed

Commit message: feat : add readme
Parts:
- added H101: IN+, MountingHole:MountingHole_3.2mm_M3_ISO7380_Pad, F.Cu at (165.2, 125.0)
- added H102: IN-, MountingHole:MountingHole_3.2mm_M3_ISO7380_Pad, F.Cu at (175.9, 125.0)
- added H4: MountingHole_Pad, MountingHole:MountingHole_2.2mm_M2_DIN965_Pad, F.Cu at (109.6, 121.2)
- added H4: MountingHole_Pad, MountingHole:MountingHole_2.2mm_M2_DIN965_Pad, F.Cu at (94.2, 138.3)
- added H4: MountingHole_Pad, MountingHole:MountingHole_2.2mm_M2_DIN965_Pad, F.Cu at (101.7, 121.4)
- added H4: MountingHole_Pad, MountingHole:MountingHole_2.2mm_M2_DIN965_Pad, F.Cu at (124.1, 137.6)
- added H4: MountingHole_Pad, MountingHole:MountingHole_2.2mm_M2_DIN965_Pad, F.Cu at (117.4, 120.9)
- added Q6: Q_NMOS_SGD, Package_SON:VSONP-8-1EP_5x6_P1.27mm, F.Cu at (117.8, 113.7)
- added Q6: Q_NMOS_SGD, Package_SON:VSONP-8-1EP_5x6_P1.27mm, F.Cu at (117.9, 128.1)
- added Q6: Q_NMOS_SGD, Package_SON:VSONP-8-1EP_5x6_P1.27mm, F.Cu at (109.5, 113.7)
- added Q6: Q_NMOS_SGD, Package_SON:VSONP-8-1EP_5x6_P1.27mm, F.Cu at (101.8, 128.5)
- added Q6: Q_NMOS_SGD, Package_SON:VSONP-8-1EP_5x6_P1.27mm, F.Cu at (101.5, 113.6)
- added Q6: Q_NMOS_SGD, Package_SON:VSONP-8-1EP_5x6_P1.27mm, F.Cu at (109.4, 128.1)
- moved J4 102.4 mm to (-34.2, 80.6)
- moved J8 102.4 mm to (-21.7, 67.8)
- moved L1 102.4 mm to (-16.9, 51.9)
- moved C1 102.4 mm to (-63.7, 81.2)
- moved C16 102.4 mm to (-63.7, 92.7)
- moved C17 102.4 mm to (-15.8, 68.0)
- moved C18 102.4 mm to (-65.2, 59.1)
- moved C19 102.4 mm to (-65.2, 61.6)
- moved C20 102.4 mm to (-65.2, 64.1)
- moved C21 102.4 mm to (-65.2, 66.6)
- moved C22 102.4 mm to (-65.2, 69.1)
- moved C23 102.4 mm to (-65.2, 71.6)
- moved C24 102.4 mm to (-65.2, 74.1)
- moved C25 102.4 mm to (-61.2, 49.0)
- moved C26 102.4 mm to (-61.2, 51.6)
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Other:
- board text added: "J2"
