File: hardware/FOC2.kicad_sch (KiCad schematic)
At the start: 94 parts, among them J1 Conn_01x03, J2 hall, J3 复用Typec, J4 Conn_01x02, J5 Conn_01x08, J6 Conn_01x04, Q1 Q_NMOS_SGD, Q2 Q_NMOS_SGD, Q3 Q_NMOS_SGD, Q4 Q_NMOS_SGD, Q5 Q_NMOS_SGD, Q6 Q_NMOS_SGD, U10 REF3033, U2 CH340N, U3 STM32G431CBUx, U4 EG2133, U5 INA199xxDCK, U6 INA199xxDCK, U7 TPS54360DDA, U8 LM358, U9 LP5907MFX-3.3

Commit message: 修改PCB和电路图
Parts:
- removed J5: Conn_01x08, Connector_Molex:Molex_PicoBlade_53047-0810_1x08_P1.25mm_Vertical, symbol Connector_Generic:Conn_01x08
- removed R20, R22: 9.5k, Resistor_SMD:R_0603_1608Metric, symbol Device:R
- removed R21: 100, Resistor_SMD:R_0603_1608Metric, symbol Device:R
- removed U8: LM358, Package_SO:SOIC-8_3.9x4.9mm_P1.27mm, symbol Amplifier_Operational:LM358
- added C31, C32, C34, C35, C37, C39: 100nf, Capacitor_SMD:C_0603_1608Metric, symbol Device:C_Small
- added C36, C38: 10uf, Capacitor_SMD:C_0603_1608Metric, symbol Device:C_Small
- added J7: Conn_01x03, Connector_Molex:Molex_PicoBlade_53047-0310_1x03_P1.25mm_Vertical, symbol Connector_Generic:Conn_01x03
- added R13, R14: 10k, Resistor_SMD:R_0603_1608Metric, symbol Device:R
- added U1: LM321, Package_TO_SOT_SMD:SOT-23-5, symbol Amplifier_Operational:LM321
- D10, D11, D2: footprint Diode_SMD:D_SOD-523 -> Diode_SMD:D_SOD-323_HandSoldering
- R19: value 100 -> 1k
Connections:
- net +3.3V: now also C31.2, C32.2, C34.2, C35.2, C36.1, C37.1, C38.1, C39.1, R13.2, U1.5 (V+)
- net FDCAN_RX: now also J7.1 (Pin_1)
- net FDCAN_TX: now also J7.2 (Pin_2)
- net GND: now also C31.1, C32.1, C34.1, C35.1, C36.2, C37.2, C38.2, C39.2, J7.3 (Pin_3), R14.1, U1.2 (V-); no longer R19.1, U5.1 (REF), U6.1 (REF)
- net HIN_1: now also U4.4 (LIN1)
- net HIN_2: now also U4.5 (LIN2)
- net HIN_3: now also U4.6 (LIN3)
- net Ialpha: now also U5.6
- net Ibeta: now also U6.6
- net LIN_1: no longer U4.4 (LIN1)
- net LIN_2: no longer U4.5 (LIN2)
- net LIN_3: no longer U4.6 (LIN3)
- net at R19.2: now also U1.3 (-), U1.4
- net M1_ENC_A: no longer names the net of C3.2, J2.2 (Pin_2), R12.2
- net M1_ENC_B: no longer names the net of C2.2, J2.3 (Pin_3), R11.2
- net M1_ENC_Z: no longer names the net of C1.2, J2.4 (Pin_4), R10.2
- new net: R13.1, R14.2, U1.1 (+)
- new net +1.65V: R19.1, U5.1 (REF), U6.1 (REF)
Other:
- note removed: "姿态传感器"
- moved on the sheet: C28, C29, U5, U6

Commit message: 保存
Parts:
- removed C1, C2, C3: 40nf, Capacitor_SMD:C_0603_1608Metric, symbol Device:C_Small
- removed R10, R11, R12: 3.3k, Resistor_SMD:R_0603_1608Metric, symbol Device:R
Connections:
- net +3.3V: no longer J2.1 (Pin_1)
- net GND: no longer J2.5 (Pin_5)
- net SPI_CLK renamed EN1
- net SPI_MISO renamed EN2
- net SPI_MOSI renamed EN3
Other:
- moved on the sheet: J6, J7

Commit message: 保存
Parts:
- removed J2: hall, Connector_Molex:Molex_PicoBlade_53047-0510_1x05_P1.25mm_Vertical, symbol Connector_Generic_MountingPin:Conn_01x05_MountingPin
- added R10, R11: 0, Resistor_SMD:R_0603_1608Metric, symbol main_board:R
- added R12: 10k, Resistor_SMD:R_0603_1608Metric, symbol main_board:R_Small
- added U8: TJA1044GTK/3Z, Package_SON:HVSON-8-1EP_3x3mm_P0.65mm_EP1.6x2.4mm, symbol main_board:TJA1044GTK_3Z
Connections:
- net +5V: now also U8.3 (VCC)
- net FDCAN_RX: now also R11.1; no longer J7.1 (Pin_1)
- net FDCAN_TX: now also R10.1; no longer J7.2 (Pin_2)
- net GND: now also R12.1, U8.2 (GND), U8.9
- new net: R10.2, U8.1 (TXD)
- new net: R11.2, U8.4 (RXD)
- new net CANH: J7.1 (Pin_1), U8.7 (CANH)
- new net CANL: J7.2 (Pin_2), U8.6 (CANL)
- new net CAN_STB: R12.2, U8.8 (STB)
- no-connect marks 7 -> 6
Other:
- note removed: "霍尔传感器"
- moved on the sheet: C30, C4, D12, J6, J7, R23, R24, U2

Commit message: 工程重构
Parts:
- removed C10, C11, C12, C13, C14, C15, C9: 47uf, Capacitor_SMD:C_1812_4532Metric, symbol Device:C
- removed C30: 10uf, Capacitor_SMD:C_0603_1608Metric, symbol Device:C_Small
- added C1: 470uf, Capacitor_THT:CP_Radial_D10.0mm_P5.00mm, symbol FOCLibrary:C
- C16: value 47uf -> 470uf; footprint Capacitor_SMD:C_1812_4532Metric -> Capacitor_THT:CP_Radial_D10.0mm_P5.00mm; symbol Device:C -> FOCLibrary:C
- C17, C18, C19, C20, C21, C22, C23, C24, C25, C26, C27, C28, C29, C31, C32, C34, C35, C36, C37, C38, C39, C4, C5, C6, C7, C8: symbol Device:C_Small -> FOCLibrary:C_Small
- C33: symbol Device:C -> FOCLibrary:C
- D1, D3: symbol Simulation_SPICE:DIODE -> FOCLibrary:DIODE
- D10, D11, D2: footprint Diode_SMD:D_SOD-323_HandSoldering -> Diode_SMD:D_SOD-123; symbol Diode:1N914WT -> FOCLibrary:1N914WT
- D12: symbol Diode:ZMMxx -> FOCLibrary:ZMMxx
- D13: symbol Device:LED -> FOCLibrary:LED
- D4, D5, D6, D7, D8, D9: symbol Diode:1N4148 -> FOCLibrary:1N4148
- H1, H2, H3, H4: symbol Mechanical:MountingHole_Pad -> FOCLibrary:MountingHole_Pad
- J1, J7: symbol Connector_Generic:Conn_01x03 -> FOCLibrary:Conn_01x03
- J3: symbol Connector:USB_C_Receptacle_USB2.0 -> FOCLibrary:USB_C_Receptacle_USB2.0
- J4: symbol Connector_Generic:Conn_01x02 -> FOCLibrary:Conn_01x02
- J6: symbol Connector_Generic:Conn_01x04 -> FOCLibrary:Conn_01x04
- L1: symbol pspice:INDUCTOR -> FOCLibrary:INDUCTOR
- Q1, Q2, Q3, Q4, Q5, Q6: symbol Device:Q_NMOS_SGD -> FOCLibrary:Q_NMOS_SGD
- R1, R13, R14, R15, R16, R17, R18, R19, R2, R23, R24, R25, R4, R5, R7, R8: symbol Device:R -> FOCLibrary:R
- R10, R11: symbol main_board:R -> FOCLibrary:R
- R12: symbol main_board:R_Small -> FOCLibrary:R_Small
- R26: symbol Device:R_Small -> FOCLibrary:R_Small
- R3, R6, R9: value 0.0005 -> 0.001; symbol Device:R -> FOCLibrary:R
- U1: symbol Amplifier_Operational:LM321 -> FOCLibrary:LM321
- U10: symbol Reference_Voltage:REF3033 -> FOCLibrary:REF3033
- U2: symbol New_Library:CH340N -> FOCLibrary:CH340N
- U3: symbol MCU_ST_STM32G4:STM32G431CBUx -> FOCLibrary:STM32G431CBUx
- U4: symbol User:EG2133 -> FOCLibrary:EG2133
- U5, U6: symbol Amplifier_Current:INA199xxDCK -> FOCLibrary:INA199xxDCK
- U7: symbol Regulator_Switching:TPS54360DDA -> FOCLibrary:TPS54360DDA
- U8: symbol main_board:TJA1044GTK_3Z -> FOCLibrary:TJA1044GTK_3Z
- U9: symbol Regulator_Linear:LP5907MFX-3.3 -> FOCLibrary:LP5907MFX-3.3
Connections:
- net GND: now also C1.2
- net VDC: now also C1.1
Other:
- moved on the sheet: C16, D12, D5, D7, D9, J1, Q2, Q4, Q6, R10, R11, R12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

Commit message: 添加驱动设计
Parts:
- removed C4: 100nf, Capacitor_SMD:C_0603_1608Metric, symbol FOCLibrary:C_Small
- removed D1: ${SIM.PARAMS}, Diode_SMD:D_SMA, symbol FOCLibrary:DIODE
- removed J3: 复用Typec, Connector_USB:USB_C_Receptacle_HRO_TYPE-C-31-M-12, symbol FOCLibrary:USB_C_Receptacle_USB2.0
- removed J7: Conn_01x03, Connector_Molex:Molex_PicoBlade_53047-0310_1x03_P1.25mm_Vertical, symbol FOCLibrary:Conn_01x03
- removed U2: CH340N, Package_SO:SOP-8_3.9x4.9mm_P1.27mm, symbol FOCLibrary:CH340N
- added J2: Conn_01x02, Connector_Molex:Molex_KK-254_AE-6410-02A_1x02_P2.54mm_Vertical, symbol FOCLibrary:Conn_01x02
- added J8: Conn_01x03, Connector_PinHeader_2.54mm:PinHeader_1x03_P2.54mm_Vertical, symbol FOCLibrary:Conn_01x03
- added J9: Conn_01x04, Connector_PinHeader_2.54mm:PinHeader_1x04_P2.54mm_Vertical, symbol FOCLibrary:Conn_01x04
- added R20, R22, R27, R28, R29: 10k, Resistor_SMD:R_0603_1608Metric, symbol FOCLibrary:R
- added R21: 120, Resistor_SMD:R_0603_1608Metric, symbol FOCLibrary:R_Small
- J6: footprint Connector_Molex:Molex_PicoBlade_53047-0410_1x04_P1.25mm_Vertical -> Connector_PinHeader_2.54mm:PinHeader_1x04_P2.54mm_Vertical
- R10, R11: value 0 -> 10k
Connections:
- net CANH: now also J2.1 (Pin_1), R21.1
- net CANL: now also J2.2 (Pin_2), R21.2
- net FDCAN_RX: now also U8.4 (RXD); no longer R11.1
- net FDCAN_TX: now also U8.1 (TXD); no longer R10.1
- net GND: now also J8.3 (Pin_3), R20.1; no longer H1.1, H2.1, H3.1, H4.1, U3.46 (PB8)
- net M1_SL_A: now also R11.2
- net M1_SL_B: now also R29.2
- net M1_SL_C: now also R28.2
- net UART_RX: now also J8.2 (Pin_2)
- net UART_TX: now also J8.1 (Pin_1)
- net VREF: no longer U3.19 (PB2)
- net VS1: now also R10.2
- net VS2: now also R22.2
- net VS3: now also R27.2
- net at D5.2 (A), Q2.2 (G), R2.2: now also R11.1
- net at D6.2 (A), Q3.2 (G), R4.2: now also R22.1
- net at D4.2 (A), Q1.2 (G), R1.2: now also R10.1
- net at D8.2 (A), Q5.2 (G), R7.2: now also R27.1
- net at D9.2 (A), Q6.2 (G), R8.2: now also R28.1
- net at D7.2 (A), Q4.2 (G), R5.2: now also R29.1
- net EN1: no longer names the net of U3.41 (PB3)
- net EN2: no longer names the net of U3.42 (PB4)
- net EN3: no longer names the net of U3.43 (PB5)
- new net: R20.2, U3.46 (PB8)
- new net Earth: H1.1, H2.1, H3.1, H4.1
- no-connect marks 6 -> 1
Other:
- note added: "通信接口"
- note removed: "通信部分"
- moved on the sheet: D12, J6, R12, R23, R24, U8
