File: hardware/FOC2.kicad_sch (KiCad schematic)
At the start: 95 parts, among them J1 Conn_01x03, J2 Conn_01x02, J4 Conn_01x02, J6 Conn_01x04, J8 Conn_01x03, J9 Conn_01x04, Q1 Q_NMOS_SGD, Q2 Q_NMOS_SGD, Q3 Q_NMOS_SGD, Q4 Q_NMOS_SGD, Q5 Q_NMOS_SGD, Q6 Q_NMOS_SGD, U1 LM321, U10 REF3033, U3 STM32G431CBUx, U4 EG2133, U5 INA199xxDCK, U6 INA199xxDCK, U7 TPS54360DDA, U8 TJA1044GTK/3Z, U9 LP5907MFX-3.3

Commit message: feat : redesign
Connections:
- net +3.3V: no longer C26.1, C27.1, C28.1, C29.1, C7.1, C8.1, R13.2, U1.5 (V+), U5.3 (V+), U6.3 (V+), U9.5 (OUT)
- new net +3V3: C26.1, C27.1, C28.1, C29.1, C7.1, C8.1, R13.2, U1.5 (V+), U5.3 (V+), U6.3 (V+), U9.5 (OUT)
Other:
- moved on the sheet: D12, J9, R23, R24, R6

Commit message: feat : add readme
Parts:
- removed C5, C8: 10uf, Capacitor_SMD:C_0603_1608Metric, symbol FOCLibrary:C_Small
- removed C6: 100nf, Capacitor_SMD:C_0603_1608Metric, symbol FOCLibrary:C_Small
- removed C7: 22nf, Capacitor_SMD:C_0603_1608Metric, symbol FOCLibrary:C_Small
- removed D4, D5, D6, D7, D8, D9: 1N4148, Diode_SMD:D_SOD-123, symbol FOCLibrary:1N4148
- removed J4: Conn_01x02, Connector_AMASS:AMASS_XT30PW-F_1x02_P2.50mm_Horizontal, symbol FOCLibrary:Conn_01x02
- removed J9: Conn_01x04, Connector_PinHeader_2.54mm:PinHeader_1x04_P2.54mm_Vertical, symbol FOCLibrary:Conn_01x04
- removed R12: 10k, Resistor_SMD:R_0603_1608Metric, symbol FOCLibrary:R_Small
- removed R21: 120, Resistor_SMD:R_0603_1608Metric, symbol FOCLibrary:R_Small
- removed U10: REF3033, Package_TO_SOT_SMD:SOT-23, symbol FOCLibrary:REF3033
- removed U8: TJA1044GTK/3Z, Package_SON:HVSON-8-1EP_3x3mm_P0.65mm_EP1.6x2.4mm, symbol FOCLibrary:TJA1044GTK_3Z
- removed U9: LP5907MFX-3.3, Package_TO_SOT_SMD:SOT-23-5, symbol FOCLibrary:LP5907MFX-3.3
- added C303, C314: 10uF, Capacitor_SMD:C_0603_1608Metric, symbol Device:C_Small
- added C305, C316: 100nF, Capacitor_SMD:C_0402_1005Metric, symbol Device:C_Small
- added H101: IN+, MountingHole:MountingHole_3.2mm_M3_ISO7380_Pad, symbol FOCLibrary:MountingHole_Pad
- added H102: IN-, MountingHole:MountingHole_3.2mm_M3_ISO7380_Pad, symbol FOCLibrary:MountingHole_Pad
- added J?: Conn_01x08, symbol Connector_Generic:Conn_01x08
- added R201: 10K, Resistor_SMD:R_0402_1005Metric, symbol Device:R
- added R203: 22, Resistor_SMD:R_0402_1005Metric, symbol Device:R
- added U301, U304: INA226, Package_SO:VSSOP-10_3x3mm_P0.5mm, symbol Sensor_Energy:INA226
- added U? (x2): ~, symbol User:TODO
- added Y201: ASCO, Crystal:Crystal_SMD_3225-4Pin_3.2x2.5mm, symbol Oscillator:ASCO
- C1, C16: value 470uf -> 47uF
- C33: value 0.1u -> 100nF
Connections:
- net VREF is gone; now on net +3.3V: U3.20 (VREF+)
- net +3.3V: now also C17.2, L1.2, R15.2, C303.1, C305.1, C314.1, C316.1, R201.1, U301.6 (VS), U304.2 (A0), U304.6 (VS), Y201.4 (VDD)
- net +5V: no longer C17.2, L1.2, R15.2
- net GND: now also C303.2, C305.2, C314.2, C316.2, H102.1, U301.1 (A1), U301.2 (A0), U301.7 (GND), U304.1 (A1), U304.7 (GND), Y201.2 (GND)
- net VDC: now also H101.1
- net at U3.5 (PF0): now also R203.1
- new net: R201.2, Y201.1 (Tri-State)
- new net: R203.2, Y201.3 (OUT)
- new net +7.5V: U304.8 (Vbus)
- new net 3.7V: U301.8 (Vbus)
- new net 3.7_ALART: U301.3 (~{Alert})
- new net 3.7_in+: U301.10 (Vin+)
- new net 3.7_in-: U301.9 (Vin-)
- new net 7.5_ALART: U304.3 (~{Alert})
- new net 7.5_in+: U304.10 (Vin+)
- new net 7.5_in-: U304.9 (Vin-)
- new net I2C_SCL: U301.5 (SCL), U304.5 (SCL)
- new net I2C_SDA: U301.4 (SDA), U304.4 (SDA)
Other:
- note added: "CAN"
- moved on the sheet: C1, C16
