File: hardware/foc-drive/FOC2.kicad_sch (KiCad schematic)
At the start: 121 parts, among them J1 Conn_02x12_Counter_Clockwise, Q1 Q_NMOS_SGD, Q2 Q_NMOS_SGD, Q3 Q_NMOS_SGD, Q4 Q_NMOS_SGD, Q5 Q_NMOS_SGD, Q6 Q_NMOS_SGD, U1 INA240A2PW, U10 SY8303, U11 TMP235A2DBZR, U12 STM32G473RCTx, U2 INA240A2PW, U3 UCC27211D, U4 UCC27211D, U5 UCC27211D, U6 INA240A2PW, U7 ME6211C33M5, U8 TCAN1044A-Q1, U9 TPS61170, Y1 ASCO

Commit message: feat: complete pcb layout
Parts:
- removed J1: Conn_02x12_Counter_Clockwise, Connector_PinHeader_2.54mm:PinHeader_2x11_P2.54mm_Vertical, symbol Connector_Generic:Conn_02x12_Counter_Clockwise
- added J1: Conn_02x12_Odd_Even, Connector_PinHeader_2.54mm:PinHeader_2x12_P2.54mm_Vertical, symbol Connector_Generic:Conn_02x12_Odd_Even
Connections:
- net CAN_H is gone; now on net CANH: L1.3
- net CAN_L is gone; now on net CANL: L1.4
- net +3.3V: now also J1.23 (Pin_23)
- net +5V: now also J1.24 (Pin_24)
- net CANH: now also J1.1 (Pin_1)
- net CANL: now also J1.3 (Pin_3)
- net ENC_A: now also J1.19 (Pin_19)
- net ENC_B: now also J1.21 (Pin_21)
- net ENC_CS: now also J1.2 (Pin_2)
- net GND: now also J1.10 (Pin_10), J1.11 (Pin_11), J1.17 (Pin_17), J1.18 (Pin_18), J1.22 (Pin_22), J1.5 (Pin_5)
- net HALL_U: now also J1.12 (Pin_12)
- net HALL_V: now also J1.14 (Pin_14)
- net HALL_W: now also J1.16 (Pin_16)
- net SPI_MISO: now also J1.6 (Pin_6)
- net SPI_MOSI: now also J1.8 (Pin_8)
- net SPI_SCK: now also J1.4 (Pin_4)
- net SWCLK: now also J1.7 (Pin_7)
- net SWDIO: now also J1.9 (Pin_9)
- net TIM1_BKIN: now also J1.20 (Pin_20)
- net UART_RX: now also J1.15 (Pin_15)
- net UART_TX: now also J1.13 (Pin_13)
- net VS1: no longer C5.1, U5.4 (HS)
- net VS3: now also C5.1, U5.4 (HS)
- net SW1: now reaches D2.2 (A), L2.2, U9.4 (SW)
- net SW2: now reaches C32.1, L3.1, U10.6 (LX)
- removed net Earth: H1.1, H2.1, H3.1, H4.1
- no-connect marks 0 -> 4
Other:
- moved on the sheet: R19

Commit message: feat: add ex pcb
Parts:
- R1, R10, R11, R17, R18, R2, R30, R31, R32, R33, R34, R35, R36, R37, R38, R5, R6: value 22 -> 10
Changed lines of the file:
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@@
 			)
 		)
-		(property "Value" "22"
+		(property "Value" "10"
 			(at 360.426 57.15 90)
 			(effects
@@
 			)
 		)
-		(property "Value" "22"
+		(property "Value" "10"
 			(at 177.165 142.875 90)
 			(effects
@@
 			)
 		)
-		(property "Value" "22"
+		(property "Value" "10"
 			(at 360.426 52.324 90)
 			(effects
@@
 			)
 		)
-		(property "Value" "22"
+		(property "Value" "10"
 			(at 137.16 165.1 90)
 			(effects
@@
 			)
 		)
-		(property "Value" "22"
+		(property "Value" "10"
 			(at 213.995 142.875 90)
 			(effects
@@
 			)
 		)
-		(property "Value" "22"
+		(property "Value" "10"
 			(at 313.436 82.55 90)
 			(effects
@@
 			)
 		)
-		(property "Value" "22"
+		(property "Value" "10"
 			(at 153.543 213.106 90)
 			(effects
@@
 			)
 		)
-		(property "Value" "22"
+		(property "Value" "10"
 			(at 313.436 85.09 90)
 			(effects
@@
 			)
 		)
-		(property "Value" "22"
+		(property "Value" "10"
 			(at 360.426 108.204 90)
 			(effects
@@
 			)
 		)
-		(property "Value" "22"
+		(property "Value" "10"
 			(at 177.165 165.1 90)
 			(effects
@@
 			)
 		)
-		(property "Value" "22"
+		(property "Value" "10"
 			(at 137.16 142.875 90)
 			(effects
@@
 			)
 		)
-		(property "Value" "22"
+		(property "Value" "10"
 			(at 313.436 80.264 90)
 			(effects
@@
 			)
 		)
-		(property "Value" "22"
+		(property "Value" "10"
 			(at 360.426 54.61 90)
 			(effects
@@
 			)
 		)
-		(property "Value" "22"
+		(property "Value" "10"
 			(at 360.426 113.03 90)
 			(effects
@@
 			)
 		)
-		(property "Value" "22"
+		(property "Value" "10"
 			(at 153.289 205.486 90)
 			(effects
@@
 			)
 		)
-		(property "Value" "22"
+		(property "Value" "10"
 			(at 360.426 110.49 90)
 			(effects
@@
 			)
 		)
-		(property "Value" "22"
+		(property "Value" "10"
 			(at 213.995 165.1 90)
 			(effects
