File: hardware/foc-drive/FOC2.kicad_pcb (KiCad board)
At the start: 2 copper layers, 50 x 72 mm, 121 parts, among them J1 Conn_02x12_Counter_Clockwise, Q1 Q_NMOS_SGD, Q2 Q_NMOS_SGD, Q3 Q_NMOS_SGD, Q4 Q_NMOS_SGD, Q5 Q_NMOS_SGD, Q6 Q_NMOS_SGD, U1 INA240A2PW, U10 SY8303, U11 TMP235A2DBZR, U12 STM32G473RCTx, U2 INA240A2PW, U3 UCC27211D, U4 UCC27211D, U5 UCC27211D, U6 INA240A2PW, U7 ME6211C33M5, U8 TCAN1044A-Q1, U9 TPS61170, Y1 ASCO

Commit message: feat: complete pcb layout
Parts:
- added REF**: ESD-Logo_6.6x6mm_SilkScreen, Symbol:ESD-Logo_6.6x6mm_SilkScreen, F.Cu at (132.7, 94.1)
- C35, U11: moved to F.Cu
- J1: value Conn_02x12_Counter_Clockwise -> Conn_02x12_Odd_Even; footprint Connector_PinHeader_2.54mm:PinHeader_2x11_P2.54mm_Vertical -> Connector_PinHeader_2.54mm:PinHeader_2x12_P2.54mm_Vertical
- moved C37 108.2 mm to (129.4, 111.5), turned to 90 degrees
- moved C38 95.6 mm to (115.2, 109.5)
- moved C39 94.8 mm to (115.2, 111.0)
- moved C36 91.8 mm to (127.9, 111.5), turned to 90 degrees
- moved R5 88.4 mm to (115.2, 107.9), turned to 180 degrees
- moved R6 86.0 mm to (115.2, 106.3), turned to 180 degrees
- moved C40 83.0 mm to (117.6, 95.3), turned to -45 degrees
- moved C41 81.4 mm to (118.7, 94.2), turned to 135 degrees
- moved R23 74.8 mm to (134.5, 70.5), turned to -90 degrees
- moved R8 73.5 mm to (133.4, 111.5), turned to -90 degrees
- moved R22 71.9 mm to (134.6, 57.7), turned to -90 degrees
- moved R9 70.7 mm to (135.0, 111.5), turned to 90 degrees
- moved C28 69.1 mm to (131.8, 111.5), turned to 90 degrees
- moved R27 68.9 mm to (99.0, 111.3), turned to 180 degrees
- moved R14 66.0 mm to (124.4, 70.7), turned to -90 degrees
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Connections:
- net Net-(D2-A) renamed /SW1
- net Net-(U10-LX) renamed /SW2
- C5 pad 1: /VS1 -> /VS3
- H1 pad 1: Earth -> unconnected-(H1-Pad1)
- H2 pad 1: Earth -> unconnected-(H2-Pad1)
- H3 pad 1: Earth -> unconnected-(H3-Pad1)
- H4 pad 1: Earth -> unconnected-(H4-Pad1)
- J1 pad 10: /ENC_A -> GND
- J1 pad 11: /ENC_B -> GND
- J1 pad 12: +3.3V -> /HALL_U
- J1 pad 13: +5V -> /UART_TX
- J1 pad 14: GND -> /HALL_V
- J1 pad 15: /TIM1_BKIN -> /UART_RX
- J1 pad 16: GND -> /HALL_W
- J1 pad 17: /HALL_W -> GND
- J1 pad 18: /HALL_V -> GND
- J1 pad 19: /HALL_U -> /ENC_A
- J1 pad 2: /CANL -> /ENC_CS
- J1 pad 20: GND -> /TIM1_BKIN
- J1 pad 21: /SPI_MOSI -> /ENC_B
- J1 pad 22: /SPI_MISO -> GND
- J1 pad 3: GND -> /CANL
- J1 pad 4: /SWCLK -> /SPI_SCK
- J1 pad 5: /SWDIO -> GND
- J1 pad 6: GND -> /SPI_MISO
- J1 pad 7: /UART_TX -> /SWCLK
- J1 pad 8: /UART_RX -> /SPI_MOSI
- J1 pad 9: GND -> /SWDIO
- L1 pad 3: /CAN_H -> /CANH
- L1 pad 4: /CAN_L -> /CANL
- U5 pad 4: /VS1 -> /VS3
Routing:
- net +3.3V: track 0.00 -> 234.7 mm, vias 0 -> 15
- net GND: track 0.00 -> 95.1 mm, vias 0 -> 134
- net +5V: track 0.00 -> 76.1 mm, vias 0 -> 6
- net +10V: track 0.00 -> 72.9 mm, vias 0 -> 6
- net /CANH: track 0.00 -> 49.6 mm, vias 0 -> 2
- net Net-(Q1-G): track 0.00 -> 48.5 mm, vias 0 -> 2
- net Net-(Q5-G): track 0.00 -> 47.0 mm, vias 0 -> 2
- net Net-(Q3-G): track 0.00 -> 46.7 mm, vias 0 -> 2
- net /CANL: track 0.00 -> 46.6 mm, vias 0 -> 2
- net /VS1: track 0.00 -> 34.2 mm, vias 0 -> 46
- net /Ialpha: track 0.00 -> 33.1 mm, vias 0 -> 2
- net /VS3: track 0.00 -> 32.5 mm, vias 0 -> 46
- net /VS2: track 0.00 -> 30.9 mm, vias 0 -> 46
- net /HIN_3: track 0.00 -> 30.5 mm, vias 0 -> 2
- net VDC: track 0.00 -> 27.1 mm, vias 0 -> 120
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- added copper zone on F.Cu, net +10V
- added copper zone on F.Cu, net +5V
- added copper zone on B.Cu, net /SAMPLE1+
- added copper zone on F.Cu, net /SAMPLE1+
- added copper zone on B.Cu, net /SAMPLE2+
- added copper zone on F.Cu, net /SAMPLE2+
- added copper zone on B.Cu, net /SAMPLE3+
- added copper zone on F.Cu, net /SAMPLE3+
- added copper zone on F.Cu, net /SW1
- added copper zone on F.Cu, net /SW2
- added copper zone on B.Cu, net /VS1
- added copper zone on F.Cu, net /VS1
- added copper zone on B.Cu, net /VS2
- added copper zone on F.Cu, net /VS2
- added copper zone on B.Cu, net /VS3
- added copper zone on F.Cu, net /VS3
- added copper zone on B.Cu, net GND
- added copper zone on F.Cu, net GND
- added copper zone on In1.Cu, net GND
- added copper zone on In2.Cu, net GND
- added copper zone on B.Cu, net VDC
- added copper zone on F.Cu, net VDC
Other:
- board size 50 x 72 mm -> 50 x 70 mm
- copper layers 2 -> 4
- board text added: "DesignedBy IpinZhu"
- board text added: "FOC-Drive VBus : 6V-30V(2S-7S) IBus : 50A(66A MAX)"

Commit message: feat: add ex pcb
Parts:
- moved C10 7.08 mm to (121.3, 86.2), turned to 180 degrees
- moved C13 6.95 mm to (110.1, 86.2), turned to 180 degrees
- moved C15 6.48 mm to (132.5, 86.2), turned to 180 degrees
- moved R18 4.41 mm to (137.6, 86.9), turned to 0 degrees
- moved R1 4.38 mm to (114.6, 87.5), turned to 0 degrees
- moved R11 4.28 mm to (125.9, 87.5), turned to 0 degrees
- moved C9 4.11 mm to (106.7, 86.2)
- moved C11 3.84 mm to (129.4, 86.2)
- moved C14 3.48 mm to (118.0, 86.2)
- moved U5 1.35 mm to (131.7, 89.7)
- moved U4 1.15 mm to (120.3, 89.7)
- moved C35 1.12 mm to (137.7, 92.6)
- moved U11 1.12 mm to (137.9, 89.7)
- moved U3 1.12 mm to (108.9, 89.7)
- moved C3 0.73 mm to (103.3, 89.1)
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Routing:
- net +10V: track 72.9 -> 77.7 mm
- net GND: track 95.1 -> 99.4 mm, vias 134 -> 246
- net /HIN_2: track 22.5 -> 18.3 mm
- net +3.3V: track 234.7 -> 230.8 mm, vias 15 -> 16
- net /HIN_1: track 15.2 -> 11.6 mm
- net /VS2: track 30.9 -> 34.0 mm
- net /LIN_2: track 17.6 -> 15.0 mm
- net Net-(Q4-G): track 19.1 -> 20.8 mm
- net Net-(Q3-G): track 46.7 -> 48.4 mm
- net Net-(Q2-G): track 20.2 -> 21.8 mm
- net /Igamma: track 20.4 -> 18.8 mm
- net /M1_GH_A: track 3.72 -> 2.43 mm
- net /M1_GL_C: track 1.86 -> 3.08 mm
- net /TEMP: track 15.4 -> 14.2 mm
- net /Ialpha: track 33.1 -> 34.3 mm
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
Commit message: feat: change readme
Parts:
- removed REF**: ESD-Logo_6.6x6mm_SilkScreen, Symbol:ESD-Logo_6.6x6mm_SilkScreen
- added G***: LOGO, LOGO, B.Cu at (104.6, 100.2)
Routing:
- net GND: vias 246 -> 249
