File: hardware/foc-drive/FOC2.kicad_pcb (KiCad board)
At the start: 4 copper layers, 50 x 70 mm, 122 parts, among them J1 Conn_02x12_Odd_Even, Q1 Q_NMOS_SGD, Q2 Q_NMOS_SGD, Q3 Q_NMOS_SGD, Q4 Q_NMOS_SGD, Q5 Q_NMOS_SGD, Q6 Q_NMOS_SGD, U1 INA240A2PW, U10 SY8303, U11 TMP235A2DBZR, U12 STM32G473RCTx, U2 INA240A2PW, U3 UCC27211D, U4 UCC27211D, U5 UCC27211D, U6 INA240A2PW, U7 ME6211C33M5, U8 TCAN1044A-Q1, U9 TPS61170, Y1 ASCO

Commit message: feat: integrate FOC host tooling and wireless control stack
- add the Vue/Tauri desktop app, device sessions and transport adapters
- add the shared v2 wire protocol and firmware control-lease handling
- replace the PlatformIO bridge with native ESP-IDF PC/motor bridges
- capture drive-board and expansion-board design updates
- document setup, simulation limits and pending board validation
- exclude KiCad recovery files and preserve local editor state

Validation: 105 firmware tests, 14 host workspace tests, 7 wire tests,
bridge C++ interface tests, frontend production build, and encoder/Hall
ARM release builds and Clippy checks passed. No board validation performed.

Co-Authored-By: Claude Fable 5 <noreply@anthropic.com>
Parts:
- added REF**: ESD-Logo_6.6x6mm_SilkScreen, Symbol:ESD-Logo_6.6x6mm_SilkScreen, B.Cu at (117.6, 93.5)
- added REF**: OSHW-Logo2_7.3x6mm_SilkScreen, Symbol:OSHW-Logo2_7.3x6mm_SilkScreen, B.Cu at (126.1, 93.0)
- moved G*** 3.74 mm to (104.9, 96.5)
Routing:
- net +3.3V: track 230.8 -> 232.4 mm
- net Net-(Q2-G): track 21.8 -> 20.7 mm
- net GND: vias 249 -> 266
Other:
- board text added: "+3.3V|B|ENC_A"
- board text added: "+5V|GND|BKIN"
- board text added: "BKIN"
- board text added: "CAN"
- board text added: "DEBUGGER"
- board text added: "ENCODER"
- board text added: "GND|CANL|CANH"
- board text added: "GND|DIO|SCK"
- board text added: "GND|MOSI|MISO|SCK|CS"
- board text added: "GND|RX|TX"
- board text added: "GND|W|V|U"
- board text added: "HALL"
- board text added: "Pin Definitions"
- board text added: "SPI"
- board text added: "U"
- board text added: "UART"
- board text added: "V"
- board text added: "Version：v1.0.0 Date：2026/9/25 Contact：github.com/IpinZhu/foc-esc.git"
- board text added: "W"
