File: hardware/foc-expansion/foc-ex.kicad_pcb (KiCad board)
At the start: 2 copper layers, 50 x 70 mm, 21 parts, among them J1 Conn_01x02, SW1 SW_Push, U1 ESP32-S3-WROOM-1, U2 ESP32-C3-WROOM-02

Commit message: feat: integrate FOC host tooling and wireless control stack
- add the Vue/Tauri desktop app, device sessions and transport adapters
- add the shared v2 wire protocol and firmware control-lease handling
- replace the PlatformIO bridge with native ESP-IDF PC/motor bridges
- capture drive-board and expansion-board design updates
- document setup, simulation limits and pending board validation
- exclude KiCad recovery files and preserve local editor state

Validation: 105 firmware tests, 14 host workspace tests, 7 wire tests,
bridge C++ interface tests, frontend production build, and encoder/Hall
ARM release builds and Clippy checks passed. No board validation performed.

Co-Authored-By: Claude Fable 5 <noreply@anthropic.com>
Parts:
- removed the C1 at (34.7, 140.4)
- removed the C1 at (57.5, 133.1)
- removed the C1 at (42.3, 140.4)
- removed the C1 at (49.9, 133.1)
- removed the C1 at (34.6, 133.0)
- removed the C1 at (42.3, 133.1)
- removed the C1 at (57.5, 140.4)
- removed the C1 at (49.9, 140.4)
- removed U2: ESP32-C3-WROOM-02, RF_Module:ESP32-C3-WROOM-02
- added C1: C_Small, Capacitor_THT:CP_Radial_D6.3mm_P2.50mm, F.Cu at (35.1, 138.3)
- added C2: C_Small, Capacitor_THT:CP_Radial_D6.3mm_P2.50mm, F.Cu at (42.9, 138.3)
- added C4: C_Small, Capacitor_THT:CP_Radial_D6.3mm_P2.50mm, F.Cu at (50.6, 138.3)
- added C6: C_Small, Capacitor_THT:CP_Radial_D6.3mm_P2.50mm, F.Cu at (58.4, 138.3)
- added J2: Conn_01x02, Connector_JST:JST_XH_B2B-XH-A_1x02_P2.50mm_Vertical, F.Cu at (66.9, 122.8)
- added SW2: SW_Push, Button_Switch_SMD:SW_Push_SPST_NO_Alps_SKRK, F.Cu at (66.0, 155.2)
- added SW3: SW_Push, Button_Switch_SMD:SW_Push_SPST_NO_Alps_SKRK, F.Cu at (66.0, 159.7)
- added SW4: SW_Push, Button_Switch_SMD:SW_Push_SPST_NO_Alps_SKRK, F.Cu at (66.0, 164.2)
- H1: value MountingHole_Pad -> IN+
- H1: renamed from ?; value (none) -> IN+
- H2: value MountingHole_Pad -> IN-
- J1: value Conn_01x02 -> Conn_02x12_Odd_Even
- SW1: footprint Button_Switch_THT:SW_PUSH_6mm -> Button_Switch_SMD:SW_Push_SPST_NO_Alps_SKRK
- U1: moved to B.Cu
- moved SW1 83.4 mm to (66.2, 149.6)
- moved U1 0.36 mm to (28.8, 157.1), turned to -90 degrees
- renumbered H6 to H2
Connections:
- H1 pad 1: unconnected-(H1-Pad1) -> VDC
- H2 pad 1: unconnected-(H2-Pad1) -> GND
- J1 pad 1: unconnected-(J1-Pin_1-Pad1) -> /CANH
- J1 pad 10: (no net) -> GND
- J1 pad 11: (no net) -> GND
- J1 pad 12: (no net) -> /HALL_U
- J1 pad 13: (no net) -> /UART_TX
- J1 pad 14: (no net) -> /HALL_V
- J1 pad 15: (no net) -> /UART_RX
- J1 pad 16: (no net) -> /HALL_W
- J1 pad 17: (no net) -> GND
- J1 pad 18: (no net) -> GND
- J1 pad 19: (no net) -> /ENC_A
- J1 pad 2: unconnected-(J1-Pin_2-Pad2) -> /ENC_CS
- J1 pad 20: (no net) -> /TIM1_BKIN
- J1 pad 21: (no net) -> /ENC_B
- J1 pad 22: (no net) -> GND
- J1 pad 23: (no net) -> +3.3V
- J1 pad 24: (no net) -> +5V
- J1 pad 3: (no net) -> /CANL
- J1 pad 4: (no net) -> /SPI_SCK
- J1 pad 5: (no net) -> GND
- J1 pad 6: (no net) -> /SPI_MISO
- J1 pad 7: (no net) -> /SWCLK
- J1 pad 8: (no net) -> /SPI_MOSI
- J1 pad 9: (no net) -> /SWDIO
- U1 pad 1: Net-(U1-GND-Pad1) -> GND
- U1 pad 2: unconnected-(U1-3V3-Pad2) -> +3.3V
- U1 pad 40: Net-(U1-GND-Pad1) -> GND
- U1 pad 41: Net-(U1-GND-Pad1) -> GND
Other:
- outline, holes or cut-outs redrawn
